File: pcb/pubmarine-submarine.kicad_pcb (KiCad board)
At the start: 2 copper layers, 100 x 80 mm, 102 parts, among them J1 Screw_Terminal_01x02, J10 Conn_01x02, J11 Conn_01x02, J12 Screw_Terminal_01x02, J13 Conn_01x03, J14 Conn_01x04, J15 Servo1, J16 Servo2, J17 Servo3, J18 Servo4, J19 Conn_01x02, J2 Conn_01x02, J20 Conn_01x02, J21 Conn_01x02, J22 Conn_01x02, J23 Conn_01x02, J24 Conn_01x02, J25 Conn_01x20, J26 Conn_01x20, J27 Conn_01x03, J3 Conn_01x02, J4 Conn_01x02, J5 Conn_01x02, J6 Screw_Terminal_01x02, J7 Screw_Terminal_01x02, J8 Conn_01x02, J9 Conn_01x02, Q1 AO3400A, Q2 AO3400A, Q3 AO3400A, Q4 AO3400A, Q5 AO3400A, Q6 AO3400A, Q7 AO3400A, Q8 AO3400A, SW1 SW_SPDT, SW2 SW_SPDT, U1 Pico, U2 SN74LV1T34DBV, U3 A4950E, U4 A4950E, U5 A4950E, U6 A4950E, U7 MPU-6050

Commit message: pcb update
Parts:
- removed D15, D16: LED, LED_SMD:LED_0603_1608Metric_Pad1.05x0.95mm_HandSolder
- removed R26: 330R, Resistor_SMD:R_0603_1608Metric_Pad0.98x0.95mm_HandSolder
- removed R27: 1K, Resistor_SMD:R_0603_1608Metric_Pad0.98x0.95mm_HandSolder
- removed SW1, SW2: SW_SPDT, Button_Switch_THT:SW_Slide_SPDT_Straight_CK_OS102011MS2Q
- added JP1: Jumper_2_Bridged, Jumper:SolderJumper-2_P1.3mm_Bridged_RoundedPad1.0x1.5mm, F.Cu at (58.2, 63.0)
- D1, D2, D3, D4, D5, D6, D7, D8: value 1N5822 -> B5819W; footprint Diode_SMD:D_0603_1608Metric -> Diode_SMD:D_SOD-123
- moved D1 1.12 mm to (62.0, 112.5)
- moved D2 1.12 mm to (69.0, 112.5)
- moved D3 1.12 mm to (76.0, 112.5)
- moved D4 1.12 mm to (83.0, 112.5)
- moved D5 1.12 mm to (93.0, 112.5)
- moved D6 1.12 mm to (100.0, 112.5)
- moved D7 1.12 mm to (107.0, 112.5)
- moved D8 1.12 mm to (114.0, 112.5)
Connections:
- net /VBUS renamed VBUS
- J12 pad 1: /PI_PWR -> +5VL
- J23 pad 1: /LED_PWR -> +12V
- J24 pad 1: /LED_PWR -> +12V
- J26 pad 2: +5VL -> Net-(J26-Pin_2)
- U1 pad 39: +5VL -> Net-(J26-Pin_2)
Routing:
- net /LED_PWR: track 24.8 -> 0.00 mm
- net /PI_PWR: track 21.7 -> 0.00 mm
- net +12V: track 155.0 -> 172.1 mm
- net Net-(J26-Pin_2): track 0.00 -> 12.0 mm
- net Net-(D16-A): track 2.05 -> 0.00 mm
- net Net-(D15-A): track 2.03 -> 0.00 mm
- net +5VL: track 195.3 -> 193.9 mm
- net +5VP: track 292.6 -> 293.8 mm

Commit message: pcb update
Routing:
- net IN_Z1: track 22.3 -> 22.8 mm
- net IN_Y2: track 21.5 -> 22.1 mm
Changed lines of the file:
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@@
 	)
 	(segment
-		(start 69.135 61.56131)
-		(end 75.02169 67.448)
+		(start 74.977849 67.448)
+		(end 84.368 67.448)
 		(width 0.25)
 		(layer "F.Cu")
@@
 	)
 	(segment
-		(start 75.02169 67.448)
-		(end 84.368 67.448)
-		(width 0.25)
-		(layer "F.Cu")
-		(net 14)
-	)
-	(segment
-		(start 69.135 60.28)
-		(end 69.135 61.56131)
+		(start 69.135 61.605151)
+		(end 74.977849 67.448)
 		(width 0.25)
 		(layer "F.Cu")
@@
 	)
 	(segment
+		(start 85.92 74.1)
+		(end 85.91 74.11)
+		(width 0.25)
+		(layer "F.Cu")
+		(net 14)
+	)
+	(segment
+		(start 69.135 60.28)
+		(end 69.135 61.605151)
+		(width 0.25)
+		(layer "F.Cu")
+		(net 14)
+	)
+	(segment
 		(start 84.368 67.448)
 		(end 85.92 69)
@@
 	)
 	(segment
-		(start 85.92 74.1)
-		(end 85.91 74.11)
-		(width 0.25)
-		(layer "F.Cu")
-		(net 14)
+		(start 77.5875 62.0875)
+		(end 77.5875 60.28)
+		(width 0.25)
+		(layer "F.Cu")
+		(net 15)
+	)
+	(segment
+		(start 88.694 66.694)
+		(end 82.194 66.694)
+		(width 0.25)
+		(layer "F.Cu")
+		(net 15)
 	)
 	(segment
@@
 	)
 	(segment
-		(start 82.26769 66.694)
+		(start 91 69)
 		(end 88.694 66.694)
-		(width 0.25)
-		(layer "F.Cu")
-		(net 15)
-	)
-	(segment
-		(start 77.5875 62.01381)
-		(end 82.26769 66.694)
-		(width 0.25)
-		(layer "F.Cu")
-		(net 15)
-	)
-	(segment
-		(start 88.694 66.694)
-		(end 91 69)
-		(width 0.25)
-		(layer "F.Cu")
-		(net 15)
-	)
-	(segment
-		(start 77.5875 60.28)
-		(end 77.5875 62.01381)
 		(width 0.25)
 		(layer "F.Cu")
@@
 	)
 	(segment
-		(start 82.071 67.071)
+		(start 82.194 66.694)
+		(end 77.5875 62.0875)
+		(width 0.25)
+		(layer "F.Cu")
+		(net 15)
+	)
+	(segment
+		(start 76.3175 62.3175)
+		(end 76.3175 60.28)
+		(width 0.25)
+		(layer "F.Cu")
+		(net 16)
+	)
+	(segment
+		(start 88.46 69)
 		(end 86.531 67.071)
 		(width 0.25)
@@
 	)
 	(segment
-		(start 76.3175 60.28)
-		(end 76.3175 61.3175)
-		(width 0.25)
-		(layer "F.Cu")
-		(net 16)
-	)
-	(segment
-		(start 76.3175 61.3175)
-		(end 82.071 67.071)
-		(width 0.25)
-		(layer "F.Cu")
-		(net 16)
-	)
-	(segment
 		(start 86.531 67.071)
-		(end 88.46 69)
+		(end 81.071 67.071)
 		(width 0.25)
 		(layer "F.Cu")
@@
 	)
 	(segment
-		(start 86.135 62.06131)
-		(end 91.180111 67.106421)
+		(start 81.071 67.071)
+		(end 76.3175 62.3175)
+		(width 0.25)
+		(layer "F.Cu")
+		(net 16)
+	)
+	(segment
+		(start 86.135 63.06727)
+		(end 90.174151 67.106421)
 		(width 0.25)
 		(layer "F.Cu")
@@
 	)
 	(segment
-		(start 91.180111 67.106421)
+		(start 90.174151 67.106421)
 		(end 96.726421 67.106421)
 		(width 0.25)
@@
 	(segment
 		(start 86.135 60.28)
-		(end 86.135 62.06131)
+		(end 86.135 63.06727)
 		(width 0.25)
 		(layer "F.Cu")
@@
 	)
 	(segment
-		(start 55.43 90.57)
-		(end 57 89)
-		(width 0.25)
-		(layer "F.Cu")
-		(net 19)
-	)
-	(segment
-		(start 55.43 91.89)
+		(start 102.335 68.513299)
+		(end 102.335 75.275)
+		(width 0.25)
+		(layer "F.Cu")
+		(net 19)
+	)
+	(segment
+		(start 57 89)
 		(end 55.43 90.57)
 		(width 0.25)
@@
 	)
 	(segment
-		(start 57 89)
-		(end 88.61 89)
+		(start 94.635 60.28)
+		(end 94.635 62.105151)
+		(width 0.25)
+		(layer "F.Cu")
+		(net 19)
+	)
+	(segment
+		(start 99.029849 66.5)
+		(end 100.321701 66.5)
 		(width 0.25)
 		(layer "F.Cu")
@@
 	)
 	(segment
-		(start 102.335 68.513299)
-		(end 100.321701 66.5)
+		(start 55.43 90.57)
+		(end 55.43 91.89)
+		(width 0.25)
+		(layer "F.Cu")
+		(net 19)
+	)
+	(segment
+		(start 102.335 75.275)
+		(end 88.61 89)
+		(width 0.25)
+		(layer "F.Cu")
+		(net 19)
+	)
+	(segment
+		(start 94.635 62.105151)
+		(end 99.029849 66.5)
+		(width 0.25)
+		(layer "F.Cu")
+		(net 19)
+	)
+	(segment
+		(start 88.61 89)
+		(end 57 89)
 		(width 0.25)
 		(layer "F.Cu")
@@
 	(segment
 		(start 100.321701 66.5)
-		(end 99.07369 66.5)
-		(width 0.25)
-		(layer "F.Cu")
-		(net 19)
-	)
-	(segment
-		(start 94.635 62.06131)
-		(end 94.635 60.28)
-		(width 0.25)
-		(layer "F.Cu")
-		(net 19)
-	)
-	(segment
-		(start 88.61 89)
-		(end 102.335 75.275)
-		(width 0.25)
-		(layer "F.Cu")
-		(net 19)
-	)
-	(segment
-		(start 99.07369 66.5)
-		(end 94.635 62.06131)
-		(width 0.25)
-		(layer "F.Cu")
-		(net 19)
-	)
-	(segment
-		(start 102.335 75.275)
 		(end 102.335 68.513299)
 		(width 0.25)
@@
 	)
 	(segment
-		(start 80.844 102.094)
-		(end 75.75 97)
-		(width 0.25)
-		(layer "F.Cu")
-		(net 36)
-	)
-	(segment
-		(start 82.844 102.094)
-		(end 80.844 102.094)
+		(start 82.314 102.064)
+		(end 85.75 105.5)
 		(width 0.25)
 		(layer "F.Cu")
@@
 	)
 	(segment
-		(start 86.25 105.5)
-		(end 82.844 102.094)
+		(start 85.75 105.5)
+		(end 86.25 105.5)
 		(width 0.25)
 		(layer "F.Cu")
@@
 	)
 	(segment
-		(start 78.29 97)
-		(end 83.384 102.094)
+		(start 80.814 102.064)
+		(end 82.314 102.064)
+		(width 0.25)
+		(layer "F.Cu")
+		(net 36)
+	)
+	(segment
+		(start 75.75 97)
+		(end 80.814 102.064)
+		(width 0.25)
+		(layer "F.Cu")
+		(net 36)
+	)
+	(segment
+		(start 83.354 102.064)
+		(end 78.29 97)
 		(width 0.25)
 		(layer "F.Cu")
@@
 	)
 	(segment
-		(start 83.384 102.094)
-		(end 92.844 102.094)
-		(width 0.25)
-		(layer "F.Cu")
-		(net 37)
-	)
-	(segment
-		(start 92.844 102.094)
-		(end 96.25 105.5)
+		(start 92.814 102.064)
+		(end 83.354 102.064)
 		(width 0.25)
 		(layer "F.Cu")
@@
 		(width 0.25)
 		(layer "F.Cu")
+		(net 37)
+	)
+	(segment
+		(start 96.25 105.5)
+		(end 92.814 102.064)
+		(width 0.25)
+		(layer "F.Cu")
