File: pcb/pubmarine-submarine.kicad_pcb (KiCad board)
At the start: 4 copper layers, 100 x 80 mm, 117 parts, among them J1 Screw_Terminal_01x02, J10 Conn_01x02, J11 Conn_01x02, J12 Screw_Terminal_01x02, J13 Conn_01x03, J14 Conn_01x04, J15 Servo1, J16 Servo2, J17 Servo3, J18 Servo4, J2 Conn_01x02, J22 Conn_01x04, J23 Conn_01x02, J24 Conn_01x02, J25 Conn_01x20, J26 Conn_01x20, J28 Conn_01x02, J29 Conn_01x02, J3 Conn_01x02, J4 Conn_01x02, J5 Conn_01x02, J6 Screw_Terminal_01x02, J7 Screw_Terminal_01x02, J8 Conn_01x02, J9 Conn_01x02, Q1 AO3400A, Q2 AO3400A, Q3 AO3400A, Q4 AO3400A, Q5 AO3400A, Q6 AO3400A, Q7 AO3400A, Q8 AO3400A, Q9 AO3400A, SW1 SW_Push, U1 Pico, U10 DRV8873H, U11 DRV8873H, U2 SN74LV1T34DBV, U5 ER_OLEDM0.91_1x-I2C, U7 MPU-6050, U9 ADS1015IDGS

Commit message: wip pcb
Parts:
- removed D1, D2, D3, D4, D5, D6, D7, D8: B5819W, Diode_SMD:D_SOD-123
- removed J25, J26: Conn_01x20, Connector_PinHeader_2.54mm:PinHeader_1x20_P2.54mm_Vertical
- removed Q1, Q2, Q3, Q4, Q5, Q6, Q7, Q8: AO3400A, Package_TO_SOT_SMD:SOT-23_Handsoldering
- removed R1, R10, R11, R12, R2, R3, R4, R9: 470R, Resistor_SMD:R_0603_1608Metric_Pad0.98x0.95mm_HandSolder
- removed R13, R14, R15, R16, R5, R6, R7, R8: 10k, Resistor_SMD:R_0603_1608Metric_Pad0.98x0.95mm_HandSolder
- added C27: C, Capacitor_SMD:C_0603_1608Metric_Pad1.08x0.95mm_HandSolder, F.Cu at (63.0, 112.8)
- added C28: C, Capacitor_SMD:C_0603_1608Metric_Pad1.08x0.95mm_HandSolder, F.Cu at (70.0, 112.8)
- added C29: C, Capacitor_SMD:C_0603_1608Metric_Pad1.08x0.95mm_HandSolder, F.Cu at (77.0, 112.8)
- added C30: C, Capacitor_SMD:C_0603_1608Metric_Pad1.08x0.95mm_HandSolder, F.Cu at (84.0, 112.8)
- added C31: C, Capacitor_SMD:C_0603_1608Metric_Pad1.08x0.95mm_HandSolder, F.Cu at (94.0, 112.8)
- added C32: C, Capacitor_SMD:C_0603_1608Metric_Pad1.08x0.95mm_HandSolder, F.Cu at (101.0, 112.8)
- added C33: C, Capacitor_SMD:C_0603_1608Metric_Pad1.08x0.95mm_HandSolder, F.Cu at (108.0, 112.8)
- added C34: C, Capacitor_SMD:C_0603_1608Metric_Pad1.08x0.95mm_HandSolder, F.Cu at (115.0, 112.8)
- added C35: 100N, Capacitor_SMD:C_0603_1608Metric_Pad1.08x0.95mm_HandSolder, F.Cu at (70.8, 104.0)
- added C36: 10U, Capacitor_SMD:C_0603_1608Metric_Pad1.08x0.95mm_HandSolder, F.Cu at (77.8, 104.0)
- added C37: 100N, Capacitor_SMD:C_0603_1608Metric_Pad1.08x0.95mm_HandSolder, F.Cu at (101.0, 104.0)
- added C38: 10U, Capacitor_SMD:C_0603_1608Metric_Pad1.08x0.95mm_HandSolder, F.Cu at (108.0, 104.0)
- added U3: DRV8847PWP, Package_SO:HTSSOP-16-1EP_4.4x5mm_P0.65mm_EP3.4x5mm_Mask2.46x2.31mm_ThermalVias, F.Cu at (74.2, 106.2)
- added U4: DRV8847PWP, Package_SO:HTSSOP-16-1EP_4.4x5mm_P0.65mm_EP3.4x5mm_Mask2.46x2.31mm_ThermalVias, F.Cu at (104.5, 106.2)
- J1, J12, J6, J7: footprint TerminalBlock:TerminalBlock_Altech_AK300-2_P5.00mm -> pubmarine-submarine:TerminalBlock_Altech_AK300-2_P5.00mm
- J28, J29: footprint Connector_JST:JST_XH_B2B-XH-AM_1x02_P2.50mm_Vertical -> pubmarine-submarine:TerminalBlock_Altech_AK300-2_P5.00mm
- R30, R33: value 10K -> 10k
- moved C4 80.7 mm to (108.8, 71.5), turned to 180 degrees
- moved U9 77.9 mm to (109.0, 68.7), turned to 0 degrees
- moved R31 74.6 mm to (108.7, 66.0), turned to 0 degrees
- moved R33 71.7 mm to (35.1, 114.0)
- moved J22 56.4 mm to (180.2, 96.4)
- moved U7 56.4 mm to (177.0, 69.5)
- moved U5 52.3 mm to (158.0, 54.0)
- moved D14 12.0 mm to (125.2, 57.2)
- moved R23 12.0 mm to (121.2, 57.2)
- moved J7 12.0 mm to (126.0, 47.0)
- moved J6 11.8 mm to (137.8, 47.0)
- moved D13 11.8 mm to (137.0, 57.2)
- moved R22 11.8 mm to (133.0, 57.2)
- moved R27 8.90 mm to (132.0, 106.5)
- moved C18 7.38 mm to (79.6, 54.5)
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Connections:
- C1 pad 1: +5VP -> +12V
- C2 pad 1: +5VP -> +12V
- J10 pad 1: +5VP -> /RL+
- J10 pad 2: /RL- -> GND
- J11 pad 1: +5VP -> /RR+
- J11 pad 2: /RR- -> GND
- J2 pad 1: +5VP -> /FU+
- J2 pad 2: /FU- -> GND
- J3 pad 1: +5VP -> /FD+
- J3 pad 2: /FD- -> GND
- J4 pad 1: +5VP -> /FL+
- J4 pad 2: /FL- -> GND
- J5 pad 1: +5VP -> /FR+
- J5 pad 2: /FR- -> GND
- J8 pad 1: +5VP -> /RU+
- J8 pad 2: /RU- -> GND
- J9 pad 1: +5VP -> /RD+
- J9 pad 2: /RD- -> GND
- R30 pad 2: ~{FAULT_A} -> ~{FAULT_M}
- R33 pad 2: ~{FAULT_B} -> ~{FAULT_J}
- U1 pad 2: Net-(J25-Pin_2) -> LIGHTS
- U1 pad 26: Net-(J26-Pin_15) -> unconnected-(U1-GPIO20-Pad26)
- U1 pad 27: Net-(J26-Pin_14) -> unconnected-(U1-GPIO21-Pad27)
- U1 pad 29: ~{SLEEP_B} -> ~{SLEEP_J}
- U1 pad 31: ~{FAULT_B} -> ~{FAULT_J}
- U1 pad 32: ~{SLEEP_A} -> ~{SLEEP_M}
- U1 pad 34: ~{FAULT_A} -> ~{FAULT_M}
- U1 pad 35: /ADC_VREF -> unconnected-(U1-ADC_VREF-Pad35)_1
- U1 pad 37: Net-(J26-Pin_4) -> unconnected-(U1-3V3_EN-Pad37)
- U10 pad 11: ~{SLEEP_A} -> ~{SLEEP_M}
- U10 pad 2: ~{FAULT_A} -> ~{FAULT_M}
- U11 pad 11: ~{SLEEP_B} -> ~{SLEEP_M}
- U11 pad 2: ~{FAULT_B} -> ~{FAULT_M}
Routing:
- net GND: track 94.2 -> 42.6 mm, vias 2 -> 0
- net ~{FAULT_M}: track 0.00 -> 39.0 mm, vias 0 -> 2
- net ~{SLEEP_M}: track 0.00 -> 37.1 mm, vias 0 -> 2
- net RUN: track 51.4 -> 18.5 mm
- net ~{SLEEP_B}: track 24.8 -> 0.00 mm, vias 1 -> 0
- net ~{FAULT_B}: track 22.4 -> 0.00 mm, vias 2 -> 0
- net /B1: track 19.8 -> 0.00 mm
- net ~{SLEEP_A}: track 18.6 -> 0.00 mm, vias 2 -> 0
- net ~{FAULT_A}: track 16.4 -> 0.00 mm
- net /A2: track 12.3 -> 0.00 mm
- net /B2: track 12.0 -> 0.00 mm
- net /A1: track 12.0 -> 0.00 mm
- net /DRV8873H/DVDD: track 25.7 -> 18.6 mm
- net +3.3V: track 19.8 -> 13.7 mm
- net +12V: track 22.0 -> 27.5 mm, vias 8 -> 64
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- added copper zone on B.Cu, net +12V
- added copper zone on F.Cu, net +12V
- added copper zone on B.Cu, net +5VP
- added copper zone on F.Cu, net /A1
- added copper zone on F.Cu, net /A2
- added copper zone on F.Cu, net /B1
- added copper zone on F.Cu, net /B2
- added copper zone on B.Cu, net GND
- added copper zone on F.Cu, net GND
- removed copper zone on In2.Cu, net +12V

Commit message: pcb rev2 done?
Parts:
- C18, C19, C27, C28, C29, C30, C31, C32, C33, C34: value C -> 100N
- moved U7 57.8 mm to (120.8, 82.8), turned to 180 degrees
- moved J22 55.9 mm to (124.3, 96.2), turned to -90 degrees
- moved R33 50.5 mm to (85.2, 108.5), turned to -90 degrees
- moved U5 30.1 mm to (128.8, 61.2)
- moved C1 10.0 mm to (66.0, 103.1)
- moved C35 8.50 mm to (79.2, 104.0)
- moved C37 8.50 mm to (109.5, 104.0)
- moved C2 7.50 mm to (114.2, 103.1)
- moved J23 7.00 mm to (123.0, 116.0)
- moved J24 7.00 mm to (130.0, 116.0)
- moved R27 6.67 mm to (126.0, 103.6), turned to 90 degrees
- moved R26 6.07 mm to (124.0, 103.6), turned to -90 degrees
- moved Q9 5.27 mm to (125.0, 108.8)
- moved R28 3.75 mm to (56.5, 66.8)
- moved C24 0.75 mm to (86.2, 56.0)
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Connections:
- U9 pad 4: unconnected-(U9-AIN0-Pad4) -> IPROPI_B
- U9 pad 5: unconnected-(U9-AIN1-Pad5) -> IPROPI_A
- U9 pad 6: unconnected-(U9-AIN2-Pad6) -> BAT_SENS
- U9 pad 7: unconnected-(U9-AIN3-Pad7) -> SENS1
Routing:
- net +3.3V: track 13.7 -> 240.2 mm, vias 0 -> 5
- net +5VL: track 13.6 -> 215.9 mm, vias 0 -> 4
- net SCL: track 0.00 -> 179.0 mm, vias 0 -> 2
- net SDA: track 0.00 -> 175.5 mm, vias 0 -> 1
- net ~{FAULT_J}: track 0.00 -> 108.6 mm, vias 0 -> 3
- net ~{SLEEP_J}: track 0.00 -> 104.6 mm, vias 0 -> 3
- net LED_DATA: track 0.00 -> 94.1 mm
- net LIGHTS: track 0.00 -> 78.8 mm, vias 0 -> 2
- net SV4: track 0.00 -> 58.4 mm
- net SV3: track 0.00 -> 52.1 mm
- net SENS1: track 0.00 -> 51.4 mm, vias 0 -> 2
- net SV1: track 0.00 -> 45.8 mm
- net SV2: track 0.00 -> 45.4 mm
- net RUN: track 18.5 -> 52.0 mm, vias 0 -> 2
- net +12V: track 27.5 -> 57.1 mm, vias 64 -> 128
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Other:
- board text added: "JLCJLCJLCJLC"
- board text added: "OLED"
- board text added: "RST"
- board text added: "TEMP/HUM"
- board text added: "The PubSubHub revision 2.0 by @DeltaWhy https://github.com/PubmarineSubmarine"
- board text added: "VSV"
- board text removed: "!! Remove 5V pullups !!"
- board text removed: "12V"
- board text removed: "5VP"
- board text removed: "The PubSubHub revision 2.0 by @DeltaWhy https://github.com/PubmarineSubmarine JLCJLCJLCJLC"

Commit message: pcb tweaks
Parts:
- R17, R18: value 4k7 -> 2k2
Routing:
- net +3.3V: track 240.2 -> 238.0 mm
- net LIGHTS: track 78.8 -> 80.1 mm
- net LED_DATA: track 94.1 -> 94.9 mm
- net SCL: track 179.0 -> 178.3 mm
Other:
- board text removed: "4k7"
