File: pcb/pubmarine-submarine.kicad_pcb (KiCad board)
At the start: 4 copper layers, 100 x 80 mm, 97 parts, among them J1 Screw_Terminal_01x02, J10 Conn_01x02, J11 Conn_01x02, J12 Screw_Terminal_01x02, J13 Conn_01x03, J14 Conn_01x04, J15 Servo1, J16 Servo2, J17 Servo3, J18 Servo4, J2 Conn_01x02, J22 Conn_01x04, J23 Conn_01x02, J24 Conn_01x02, J28 Conn_01x02, J29 Conn_01x02, J3 Conn_01x02, J4 Conn_01x02, J5 Conn_01x02, J6 Screw_Terminal_01x02, J7 Screw_Terminal_01x02, J8 Conn_01x02, J9 Conn_01x02, Q9 AO3400A, SW1 SW_Push, U1 Pico, U10 DRV8873H, U11 DRV8873H, U2 SN74LV1T34DBV, U3 DRV8847PWP, U4 DRV8847PWP, U5 ER_OLEDM0.91_1x-I2C, U7 MPU-6050, U9 ADS1015IDGS

Commit message: pcb updates
Parts:
- added C5: 100N, Capacitor_SMD:C_0603_1608Metric_Pad1.08x0.95mm_HandSolder, F.Cu at (144.5, 49.5)
- added C6: 100N, Capacitor_SMD:C_0603_1608Metric_Pad1.08x0.95mm_HandSolder, F.Cu at (127.7, 97.2)
- added J19: Conn_01x03_Pin, Connector_PinHeader_2.54mm:PinHeader_1x03_P2.54mm_Vertical, F.Cu at (53.0, 107.0)
- added J20: Conn_01x02_Pin, Connector_PinHeader_2.54mm:PinHeader_1x02_P2.54mm_Vertical, F.Cu at (60.2, 64.3)
- added TP1: TestPoint, TestPoint:TestPoint_Pad_D1.0mm, B.Cu at (83.5, 68.0)
- added TP2: TestPoint, TestPoint:TestPoint_Pad_D1.0mm, B.Cu at (100.5, 67.5)
- J15: value Servo1 -> Conn_01x03
- J16: value Servo2 -> Conn_01x03
- J17: value Servo3 -> Conn_01x03
- J18: value Servo4 -> Conn_01x03
- J28, J29: value Conn_01x02 -> Screw_Terminal_01x02
- R28: value 10K -> 10k
- moved C14 0.59 mm to (72.5, 55.4)
- moved C15 0.59 mm to (71.0, 55.4)
Connections:
- U1 pad 26: unconnected-(U1-GPIO20-Pad26) -> ~{SLEEP_J}
- U1 pad 27: unconnected-(U1-GPIO21-Pad27) -> ~{FAULT_J}
- U1 pad 29: ~{SLEEP_J} -> ~{SLEEP_M}
- U1 pad 31: ~{FAULT_J} -> Net-(J19-Pin_3)
- U1 pad 32: ~{SLEEP_M} -> Net-(J19-Pin_2)
- U7 pad 1: +5VL -> +3.3V
Routing:
- net Net-(J19-Pin_3): track 0.00 -> 40.9 mm, vias 0 -> 1
- net Net-(J19-Pin_2): track 0.00 -> 40.1 mm, vias 0 -> 1
- net +3.3V: track 238.0 -> 199.3 mm, vias 5 -> 4
- net +5VL: track 215.9 -> 231.0 mm, vias 4 -> 2
- net ~{FAULT_J}: track 108.6 -> 98.4 mm
- net ~{SLEEP_J}: track 104.6 -> 97.0 mm
- net RUN: track 52.0 -> 54.8 mm
- net ~{SLEEP_M}: track 36.7 -> 34.6 mm, vias 2 -> 3
- net IPROPI_A: track 33.6 -> 35.2 mm
- net IPROPI_B: track 18.9 -> 20.3 mm, vias 0 -> 1
- net +12V: track 57.1 -> 57.7 mm
- net Net-(U10-VCP): track 5.08 -> 5.69 mm
- net GND: vias 3 -> 37

Commit message: pcb update
Routing:
- net +12V: track 57.7 -> 58.9 mm
Changed lines of the file:
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@@
+	)
+	(segment
+		(start 86.25 55.1375)
+		(end 85.2375 55.1375)
+		(width 0.25)
+		(layer "F.Cu")
+		(net "+12V")
 	)
 	(segment
@@
 		(layer "F.Cu")
 		(net "+12V")
+	)
+	(segment
+		(start 85.2375 55.1375)
+		(end 85.1 55)
+		(width 0.25)
+		(layer "F.Cu")
+		(net "+12V")
