File: pcb/pubmarine-submarine.kicad_sch (KiCad schematic)
At the start: 68 parts, among them J1 GPIO_IN, J10 RPD, J11 Screw_Terminal_01x08, J12 Screw_Terminal_01x08, J13 ADC_HDR, J14 PWM_HDR, J2 GPIO_OUT, J3 FYL, J4 FYR, J5 FPU, J6 FPD, J7 RPU, J8 RYL, J9 RYR, Q1 AO3400A, Q2 AO3400A, Q3 AO3400A, Q4 AO3400A, Q5 AO3400A, Q6 AO3400A, Q7 AO3400A, Q8 AO3400A, U1 A4950E, U2 A4950E, U3 A4950E, U4 A4950E, U5 TLC5947DAP, U6 MCP3008

Commit message: new PCB
Parts:
- removed C1, C5, C7: 0.22uF, Capacitor_SMD:C_0603_1608Metric_Pad1.08x0.95mm_HandSolder, symbol Device:C
- removed C2, C4, C6, C8: 100uF, Capacitor_THT:CP_Radial_D5.0mm_P2.50mm, symbol Device:C_Polarized
- removed H1: MountingHole_Pad, MountingHole:MountingHole_3.2mm_M3_Pad, symbol Mechanical:MountingHole_Pad
- removed H4: MountingHole, MountingHole:MountingHole_3.2mm_M3, symbol Mechanical:MountingHole
- removed J1: GPIO_IN, Connector_PinHeader_2.54mm:PinHeader_2x20_P2.54mm_Vertical, symbol Connector:Raspberry_Pi_2_3
- removed J10: RPD, Connector_JST:JST_PH_B2B-PH-K_1x02_P2.00mm_Vertical, symbol Connector:Conn_01x02_Pin
- removed J11, J12: Screw_Terminal_01x08, TerminalBlock_Phoenix:TerminalBlock_Phoenix_MKDS-1,5-8_1x08_P5.00mm_Horizontal, symbol Connector:Screw_Terminal_01x08
- removed J13: ADC_HDR, Connector_PinHeader_2.54mm:PinHeader_1x08_P2.54mm_Vertical, symbol Connector:Conn_01x08_Pin
- removed J14: PWM_HDR, Connector_PinHeader_2.54mm:PinHeader_1x08_P2.54mm_Vertical, symbol Connector:Conn_01x08_Pin
- removed J2: GPIO_OUT, Connector_PinHeader_2.54mm:PinHeader_2x20_P2.54mm_Vertical, symbol Connector:Raspberry_Pi_2_3
- removed J3: FYL, Connector_JST:JST_PH_B2B-PH-K_1x02_P2.00mm_Vertical, symbol Connector:Conn_01x02_Pin
- removed J4: FYR, Connector_JST:JST_PH_B2B-PH-K_1x02_P2.00mm_Vertical, symbol Connector:Conn_01x02_Pin
- removed J5: FPU, Connector_JST:JST_PH_B2B-PH-K_1x02_P2.00mm_Vertical, symbol Connector:Conn_01x02_Pin
- removed J6: FPD, Connector_JST:JST_PH_B2B-PH-K_1x02_P2.00mm_Vertical, symbol Connector:Conn_01x02_Pin
- removed J7: RPU, Connector_JST:JST_PH_B2B-PH-K_1x02_P2.00mm_Vertical, symbol Connector:Conn_01x02_Pin
- removed J8: RYL, Connector_JST:JST_PH_B2B-PH-K_1x02_P2.00mm_Vertical, symbol Connector:Conn_01x02_Pin
- removed J9: RYR, Connector_JST:JST_PH_B2B-PH-K_1x02_P2.00mm_Vertical, symbol Connector:Conn_01x02_Pin
- removed Q1, Q2, Q3, Q4, Q5, Q6, Q7, Q8: AO3400A, Package_TO_SOT_SMD:SOT-23, symbol Transistor_FET:AO3400A
- removed U1, U2: A4950E, Package_SO:SOIC-8-1EP_3.9x4.9mm_P1.27mm_EP2.41x3.3mm, symbol Driver_Motor:A4950E
- removed U5: TLC5947DAP, Package_SO:HTSSOP-32-1EP_6.1x11mm_P0.65mm_EP5.2x11mm_Mask4.11x4.36mm_ThermalVias, symbol Driver_LED:TLC5947DAP
- removed U6: MCP3008, Package_SO:SOIC-16_3.9x9.9mm_P1.27mm, symbol Analog_ADC:MCP3008
- added C1, C11, C2, C5, C7, C9: 100uF, Capacitor_THT:CP_Radial_D6.3mm_P2.50mm, symbol Device:C_Polarized_US
- added C10, C4, C6, C8: 0.22uF, Capacitor_SMD:C_0603_1608Metric_Pad1.08x0.95mm_HandSolder, symbol Device:C
- added D10, D11, D9: WS2812B, LED_SMD:LED_WS2812B_PLCC4_5.0x5.0mm_P3.2mm, symbol LED:WS2812B
- added D12, D13, D14: LED, LED_SMD:LED_0603_1608Metric_Pad1.05x0.95mm_HandSolder, symbol Device:LED
- added H1: MountingHole, MountingHole:MountingHole_2.2mm_M2, symbol Mechanical:MountingHole
- added H4: MountingHole_Pad, MountingHole:MountingHole_2.2mm_M2_Pad, symbol Mechanical:MountingHole_Pad
- added J1, J12, J6, J7: Screw_Terminal_01x02, TerminalBlock:TerminalBlock_Altech_AK300-2_P5.00mm, symbol Connector:Screw_Terminal_01x02
- added J10, J11, J2, J23, J24, J3, J4, J5, J8, J9: Conn_01x02, Connector_JST:JST_PH_B2B-PH-K_1x02_P2.00mm_Vertical, symbol Connector_Generic:Conn_01x02
- added J13: Conn_01x03, Connector_JST:JST_PH_B3B-PH-K_1x03_P2.00mm_Vertical, symbol Connector_Generic:Conn_01x03
- added J14: Conn_01x04, Connector_JST:JST_PH_B4B-PH-K_1x04_P2.00mm_Vertical, symbol Connector_Generic:Conn_01x04
- added J15: Servo1, Connector_JST:JST_PH_B3B-PH-K_1x03_P2.00mm_Vertical, symbol Connector_Generic:Conn_01x03
- added J16: Servo2, Connector_JST:JST_PH_B3B-PH-K_1x03_P2.00mm_Vertical, symbol Connector_Generic:Conn_01x03
- added J17: Servo3, Connector_JST:JST_PH_B3B-PH-K_1x03_P2.00mm_Vertical, symbol Connector_Generic:Conn_01x03
- added J18: Servo4, Connector_JST:JST_PH_B3B-PH-K_1x03_P2.00mm_Vertical, symbol Connector_Generic:Conn_01x03
- added J19, J20, J21, J22: Conn_01x02, Connector_JST:JST_XH_B2B-XH-AM_1x02_P2.50mm_Vertical, symbol Connector_Generic:Conn_01x02
- added Q1, Q2, Q3, Q4, Q5, Q6, Q7, Q8: Q_NMOS_Depletion_DGS, Package_TO_SOT_SMD:SOT-223-3_TabPin2, symbol Device:Q_NMOS_Depletion_DGS
- added R21: 1K, Resistor_SMD:R_0603_1608Metric_Pad0.98x0.95mm_HandSolder, symbol Device:R
- added R22, R23: 330, Resistor_SMD:R_0603_1608Metric_Pad0.98x0.95mm_HandSolder, symbol Device:R
- added R24, R25: R, symbol Device:R
- added SW1, SW2, SW3: SW_SPDT, Button_Switch_THT:SW_Slide_SPDT_Straight_CK_OS102011MS2Q, symbol Switch:SW_SPDT
- added U1: Pico, MCU_RaspberryPi_and_Boards:RPi_Pico_SMD_TH, symbol MCU_RaspberryPi_and_Boards:Pico
- added U2: SN74LV1T34DBV, Package_TO_SOT_SMD:SOT-23-5, symbol Logic_LevelTranslator:SN74LV1T34DBV
- added U5, U6: A4950E, Package_SO:SOIC-8-1EP_3.9x4.9mm_P1.27mm_EP2.62x3.51mm_ThermalVias, symbol Driver_Motor:A4950E
- C3: value 0.22uF -> 0.1uF
- D1, D2, D3, D4, D5, D6, D7, D8: value D_Schottky -> 1N5822; footprint Diode_SMD:D_0603_1608Metric_Pad1.05x0.95mm_HandSolder -> Diode_SMD:D_0603_1608Metric
- H2, H3: footprint MountingHole:MountingHole_3.2mm_M3 -> MountingHole:MountingHole_2.2mm_M2
- R1, R2, R3, R4: value 1.1Ω -> 470; footprint Resistor_SMD:R_1812_4532Metric_Pad1.30x3.40mm_HandSolder -> Resistor_SMD:R_0603_1608Metric_Pad0.98x0.95mm_HandSolder
- R10, R12: value 100 -> 470
- R11, R9: value 1K -> 470
- R13, R15, R6, R7: value 1K -> 10k
- R14, R16, R5, R8: value 100 -> 10k
- R17: value 1K -> 4.7K
- R18: value 100 -> 4.7K
- R19: value 1K -> 10K
- R20: value 100 -> 20K
- U3, U4: footprint Package_SO:SOIC-8-1EP_3.9x4.9mm_P1.27mm_EP2.41x3.3mm -> Package_SO:SOIC-8-1EP_3.9x4.9mm_P1.27mm_EP2.62x3.51mm_ThermalVias
Connections:
- net GND: now also C3.2, R14.2, R16.2, R20.2, R5.2, R8.2, U3.1 (GND), U3.9 (PAD), U4.1 (GND), U4.9 (PAD), C1.2, C10.2, C11.2, C2.2, C4.2, C5.2, C6.2, C7.2, C8.2, C9.2, D10.3 (VSS), D11.3 (VSS), D12.1 (K), D13.1 (K), D14.1 (K), D9.3 (VSS), H4.1, J1.2 (Pin_2), J12.2 (Pin_2), J13.1 (Pin_1), J14.1 (Pin_1), J15.1 (Pin_1), J16.1 (Pin_1), J17.1 (Pin_1), J18.1 (Pin_1), J23.2 (Pin_2), J24.2 (Pin_2), J6.2 (Pin_2), J7.2 (Pin_2), Q1.3 (S), Q2.3 (S), Q3.3 (S), Q4.3 (S), Q5.3 (S), Q6.3 (S), Q7.3 (S), Q8.3 (S), R25.2, U1.13 (GND), U1.18 (GND), U1.23 (GND), U1.28 (GND), U1.3 (GND), U1.33 (AGND), U1.38 (GND), U1.42 (GND), U1.8 (GND), U2.3 (GND), U5.1 (GND), U5.9 (PAD), U6.1 (GND), U6.9 (PAD); no longer R11.2, R17.2, R19.2, R9.2
- net W+: now also J22.1 (Pin_1), U6.6 (OUT1)
- net W-: now also J22.2 (Pin_2), U6.8 (OUT2)
- net X+: now also J19.1 (Pin_1); no longer U4.6 (OUT1)
- net X-: now also J19.2 (Pin_2); no longer U4.8 (OUT2)
- net Y+: now also U4.6 (OUT1), J20.1 (Pin_1)
- net Y-: now also U4.8 (OUT2), J20.2 (Pin_2)
- net Z+: now also J21.1 (Pin_1), U5.6 (OUT1)
- net Z-: now also J21.2 (Pin_2), U5.8 (OUT2)
- net at R12.2: now also R16.1, Q8.2 (G)
- net FD: now reaches R2.1
- net FD: now also U1.7 (GPIO5)
- net +5VL: now reaches R18.2
- net +5VL: now also C3.1, R17.2, D10.1 (VDD), D11.1 (VDD), D9.1 (VDD), J12.1 (Pin_1), J13.2 (Pin_2), J14.2 (Pin_2), R23.1, SW3.3 (C), U1.39 (VSYS), U2.5 (VCC)
- net at R10.2: now also R14.1, Q6.2 (G)
- net at U3.7 (LSS): no longer R3.1
- net IN_Y2: now reaches U4.2 (IN2)
- net IN_Y2: now also U1.25 (GPIO19)
- net IN_Y1: now reaches U4.3 (IN1)
- net IN_Y1: now also U1.24 (GPIO18)
- net at U4.7 (LSS): no longer R4.1
- net FU: now reaches R1.1
- net FU: now also U1.6 (GPIO4)
- net IN_X2: now reaches U3.2 (IN2)
- net IN_X2: now also U1.22 (GPIO17)
- net IN_X1: now reaches U3.3 (IN1)
- net IN_X1: now also U1.21 (GPIO16)
- net +12VA renamed +5VP
- net +5VP: now also C1.1, C2.1, J10.1 (Pin_1), J11.1 (Pin_1), J15.2 (Pin_2), J16.2 (Pin_2), J17.2 (Pin_2), J18.2 (Pin_2), J2.1 (Pin_1), J23.1 (Pin_1), J24.1 (Pin_1), J3.1 (Pin_1), J4.1 (Pin_1), J5.1 (Pin_1), J8.1 (Pin_1), J9.1 (Pin_1), R22.1, SW2.3 (C); no longer C3.1, U3.5 (VBB), U4.5 (VBB)
- net +3V3 renamed +3.3V
- net +3.3V: now also U1.36 (3V3), U5.4 (VREF), U6.4 (VREF)
- net FPD- renamed FR-
- net FR-: now also J5.2 (Pin_2), Q4.1 (D)
- net FPU- renamed FL-
- net FL-: now also J4.2 (Pin_2), Q3.1 (D)
- net FYL- renamed FU-
- net FU-: now also J2.2 (Pin_2), Q1.1 (D)
- net FYR- renamed FD-
- net FD-: now also J3.2 (Pin_2), Q2.1 (D)
- removed net GNDA: C3.2, R1.2, R2.2, R3.2, R4.2, U3.1 (GND), U3.9 (PAD), U4.1 (GND), U4.9 (PAD)
- net PWM10 renamed RD
- net RD: now also U1.12 (GPIO9); no longer R9.1
- net PWM11 renamed RL
- net RL: now also U1.14 (GPIO10); no longer R12.1
- net PWM12: no longer names the net of R13.1
- net PWM12: now also R9.2, Q5.2 (G); no longer R14.1
- net PWM13: no longer names the net of R15.1
- net PWM13: now also R11.2, Q7.2 (G); no longer R16.1
- net PWM14 renamed SCL
- net SCL: now also J14.4 (Pin_4), U1.5 (GPIO3); no longer R17.1
- net PWM15: no longer names the net of R19.1
- net PWM15: now also J13.3 (Pin_3); no longer R20.1
- net PWM8: no longer names the net of R6.1
- net PWM8: now also R2.2, Q2.2 (G); no longer R5.1
- net PWM9: no longer names the net of R7.1
- net PWM9: now also R3.2, Q3.2 (G); no longer R8.1
- net RPD- renamed RR-
- net RR-: now also J11.2 (Pin_2), Q8.1 (D)
- net RPU- renamed RL-
- net RL-: now also J10.2 (Pin_2), Q7.1 (D)
- net RYL- renamed RU-
- net RU-: now also J8.2 (Pin_2), Q5.1 (D)
- net RYR- renamed RD-
- net RD-: now also J9.2 (Pin_2), Q6.1 (D)
- new net: D13.2 (A), R22.2
- new net: Q4.2 (G), R4.2, R8.1
- new net: D12.2 (A), R21.2
- new net: D10.4 (DIN), D9.2 (DOUT)
- new net: D9.4 (DIN), U2.4 (Y)
- new net: J1.1 (Pin_1), SW1.2 (B)
- new net: J7.1 (Pin_1), SW3.2 (B)
- new net: J6.1 (Pin_1), SW2.2 (B)
- new net: Q1.2 (G), R1.2, R5.1
- new net: D14.2 (A), R23.2
- new net: D10.2 (DOUT), D11.4 (DIN)
- new net +12V: C10.1, C11.1, C4.1, C5.1, C6.1, C7.1, C8.1, C9.1, R21.1, R24.1, SW1.3 (C), U3.5 (VBB), U4.5 (VBB), U5.5 (VBB), U6.5 (VBB)
- new net BAT_SENS: R24.2, R25.1, U1.32 (GPIO27_ADC1)
- new net FL: R3.1, U1.9 (GPIO6)
- new net FR: R4.1, U1.10 (GPIO7)
- new net IN_W1: U1.29 (GPIO22), U6.3 (IN1)
- new net IN_W2: U1.2 (GPIO1), U6.2 (IN2)
- new net IN_Z1: U1.26 (GPIO20), U5.3 (IN1)
- new net IN_Z2: U1.27 (GPIO21), U5.2 (IN2)
- new net LED_DATA: U1.1 (GPIO0), U2.2 (A)
- new net RR: R12.1, U1.15 (GPIO11)
- new net RU: R9.1, U1.11 (GPIO8)
- new net SDA: J14.3 (Pin_3), R17.1, U1.4 (GPIO2)
- new net SENS1: R19.2, R20.1, U1.31 (GPIO26_ADC0)
- new net SV1: J15.3 (Pin_3), U1.16 (GPIO12)
- new net SV2: J16.3 (Pin_3), U1.17 (GPIO13)
- new net SV3: J17.3 (Pin_3), U1.19 (GPIO14)
- new net SV4: J18.3 (Pin_3), U1.20 (GPIO15)
- no-connect marks 2 -> 15
Other:
- note added: "Battery Voltage Sense"
- note added: "Blinkenlights"
- note added: "Bulk Capacitors"
- note added: "I2C Pullups"
- note added: "IMU Breakout"
- note added: "Microcontroller"
- note added: "Power In/Out"
- note added: "Power output for lights"
- note added: "Power output to RPi"
- note added: "Pressure Sensor"
- note added: "Sensors"
- note added: "Servos"
- note removed: "ADC"
- note removed: "Front"
- note removed: "MOSFET Drivers"
- note removed: "PWM Driver"
- note removed: "Pi GPIO Chained Output"
- note removed: "Pi GPIO Input"
- note removed: "Rear"
- note removed: "Screw Terminals"

Commit message: pcb updates
Parts:
- removed SW3: SW_SPDT, Button_Switch_THT:SW_Slide_SPDT_Straight_CK_OS102011MS2Q, symbol Switch:SW_SPDT
- added D15, D16: LED, LED_SMD:LED_0603_1608Metric_Pad1.05x0.95mm_HandSolder, symbol Device:LED
- added J25, J26: Conn_01x20, Connector_PinHeader_2.54mm:PinHeader_1x20_P2.54mm_Vertical, symbol Connector_Generic:Conn_01x20
- added J27: Conn_01x03, Connector_PinHeader_2.54mm:PinHeader_1x03_P2.54mm_Vertical, symbol Connector_Generic:Conn_01x03
- added R26: 330, Resistor_SMD:R_0603_1608Metric_Pad0.98x0.95mm_HandSolder, symbol Device:R
- added R27: 1K, Resistor_SMD:R_0603_1608Metric_Pad0.98x0.95mm_HandSolder, symbol Device:R
- R24, R25: footprint (none) -> Resistor_SMD:R_0603_1608Metric_Pad0.98x0.95mm_HandSolder
Connections:
- net +12V: now also J1.1 (Pin_1), SW2.3 (C); no longer SW1.3 (C)
- net +3.3V: now also J26.5 (Pin_5)
- net +5VL: now also J7.1 (Pin_1), SW1.3 (C), J26.2 (Pin_2); no longer J12.1 (Pin_1)
- net +5VP: now also J6.1 (Pin_1); no longer J23.1 (Pin_1), J24.1 (Pin_1), SW2.3 (C)
- net BAT_SENS: now also J26.9 (Pin_9)
- net FD: now also J25.7 (Pin_7)
- net FL: now also J25.9 (Pin_9)
- net FR: now also J25.10 (Pin_10)
- net FU: now also J25.6 (Pin_6)
- net GND: now also D15.1 (K), D16.1 (K), J25.13 (Pin_13), J25.18 (Pin_18), J25.3 (Pin_3), J25.8 (Pin_8), J26.13 (Pin_13), J26.18 (Pin_18), J26.3 (Pin_3), J26.8 (Pin_8), J27.2 (Pin_2)
- net IN_W1: now also U1.2 (GPIO1), J25.2 (Pin_2); no longer U1.29 (GPIO22)
- net IN_W2: now also U1.21 (GPIO16), J26.20 (Pin_20); no longer U1.2 (GPIO1)
- net IN_X1: now also U1.27 (GPIO21), J26.14 (Pin_14); no longer U1.21 (GPIO16)
- net IN_X2: now also U1.29 (GPIO22), J26.12 (Pin_12); no longer U1.22 (GPIO17)
- net IN_Y1: now also U1.25 (GPIO19), J26.16 (Pin_16); no longer U1.24 (GPIO18)
- net IN_Y2: now also U1.26 (GPIO20), J26.15 (Pin_15); no longer U1.25 (GPIO19)
- net IN_Z1: now also U1.22 (GPIO17), J26.19 (Pin_19); no longer U1.26 (GPIO20)
- net IN_Z2: now also U1.24 (GPIO18), J26.17 (Pin_17); no longer U1.27 (GPIO21)
- net LED_DATA: now also J25.1 (Pin_1)
- net RD: now also J25.12 (Pin_12)
- net RL: now also J25.14 (Pin_14)
- net RR: now also J25.15 (Pin_15)
- net RU: now also J25.11 (Pin_11)
- net SCL: now also J25.5 (Pin_5)
- net SDA: now also J25.4 (Pin_4)
- net SENS1: now also J26.10 (Pin_10)
- net SV1: now also U1.20 (GPIO15), J25.20 (Pin_20); no longer U1.16 (GPIO12)
- net SV2: now also U1.19 (GPIO14), J25.19 (Pin_19); no longer U1.17 (GPIO13)
- net SV3: now also U1.17 (GPIO13), J25.17 (Pin_17); no longer U1.19 (GPIO14)
- net SV4: now also U1.16 (GPIO12), J25.16 (Pin_16); no longer U1.20 (GPIO15)
- net RUN: now reaches U1.30 (RUN)
- net RUN: now also J26.11 (Pin_11)
- net GPIO28_ADC2: now reaches U1.34 (GPIO28_ADC2)
- net GPIO28_ADC2: now also J26.7 (Pin_7)
- net ADC_VREF: now reaches U1.35 (ADC_VREF)
- net ADC_VREF: now also J26.6 (Pin_6)
- net at U1.37 (3V3_EN): now also J26.4 (Pin_4)
- net VBUS: now reaches U1.40 (VBUS)
- net VBUS: now also J26.1 (Pin_1)
- net at U1.41 (SWCLK): now also J27.1 (Pin_1)
- net at U1.43 (SWDIO): now also J27.3 (Pin_3)
- net PI_PWR: now reaches SW1.2 (B)
- net PI_PWR: now also J12.1 (Pin_1), R26.1; no longer J1.1 (Pin_1)
- net LED_PWR: now reaches SW2.2 (B)
- net LED_PWR: now also J23.1 (Pin_1), J24.1 (Pin_1), R27.1; no longer J6.1 (Pin_1)
- net W+ renamed WA
- net W- renamed WB
- net X+ renamed XA
- net X- renamed XB
- net Y+ renamed YA
- net Y- renamed YB
- net Z+ renamed ZA
- net Z- renamed ZB
- new net: D16.2 (A), R27.2
- new net: D15.2 (A), R26.2
- no-connect marks 15 -> 7
Other:
- moved on the sheet: J23, J24

Commit message: pcb update
Parts:
- Q1, Q2, Q3, Q4, Q5, Q6, Q7, Q8: value Q_NMOS_Depletion_DGS -> AO3400A; footprint Package_TO_SOT_SMD:SOT-223-3_TabPin2 -> Package_TO_SOT_SMD:SOT-23_Handsoldering; symbol Device:Q_NMOS_Depletion_DGS -> Device:Q_NMOS_GSD
Connections:
- net FD-: now also Q2.3 (D); no longer Q2.1 (D)
- net FL-: now also Q3.3 (D); no longer Q3.1 (D)
- net FR-: now also Q4.3 (D); no longer Q4.1 (D)
- net FU-: now also Q1.3 (D); no longer Q1.1 (D)
- net GND: now also Q1.2 (S), Q2.2 (S), Q3.2 (S), Q4.2 (S), Q5.2 (S), Q6.2 (S), Q7.2 (S), Q8.2 (S); no longer Q1.3 (S), Q2.3 (S), Q3.3 (S), Q4.3 (S), Q5.3 (S), Q6.3 (S), Q7.3 (S), Q8.3 (S)
- net RD-: now also Q6.3 (D); no longer Q6.1 (D)
- net RL-: now also Q7.3 (D); no longer Q7.1 (D)
- net RR-: now also Q8.3 (D); no longer Q8.1 (D)
- net RU-: now also Q5.3 (D); no longer Q5.1 (D)
- net at R2.2, R6.1: now also Q2.1 (G); no longer Q2.2 (G)
- net at R12.2, R16.1: now also Q8.1 (G); no longer Q8.2 (G)
- net at R13.1, R9.2: now also Q5.1 (G); no longer Q5.2 (G)
- net at R3.2, R7.1: now also Q3.1 (G); no longer Q3.2 (G)
- net at R10.2, R14.1: now also Q6.1 (G); no longer Q6.2 (G)
- net at R4.2, R8.1: now also Q4.1 (G); no longer Q4.2 (G)
- net at R11.2, R15.1: now also Q7.1 (G); no longer Q7.2 (G)
- net at R1.2, R5.1: now also Q1.1 (G); no longer Q1.2 (G)
Changed lines of the file:
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@@
 	)
 	(symbol
-		(lib_id "Device:Q_NMOS_Depletion_DGS")
+		(lib_id "Device:Q_NMOS_GSD")
 		(at 195.58 48.26 0)
 		(unit 1)
@@
 			)
 		)
-		(property "Value" "Q_NMOS_Depletion_DGS"
+		(property "Value" "AO3400A"
 			(at 201.93 49.5299 0)
 			(effects
@@
 				)
 				(justify left)
-				(hide yes)
 			)
 		)
-		(property "Footprint" "Package_TO_SOT_SMD:SOT-223-3_TabPin2"
-			(at 195.58 48.26 0)
+		(property "Footprint" "Package_TO_SOT_SMD:SOT-23_Handsoldering"
+			(at 200.66 45.72 0)
 			(effects
 				(font
@@
 			)
 		)
-		(property "Description" "Depletion-mode N-channel MOSFET, drain/gate/source"
+		(property "Description" "N-MOSFET transistor, gate/source/drain"
 			(at 195.58 48.26 0)
 			(effects
@@
 	)
 	(symbol
-		(lib_id "Device:Q_NMOS_Depletion_DGS")
+		(lib_id "Device:Q_NMOS_GSD")
 		(at 228.6 48.26 0)
 		(unit 1)
@@
 			)
 		)
-		(property "Value" "Q_NMOS_Depletion_DGS"
+		(property "Value" "AO3400A"
 			(at 234.95 49.5299 0)
 			(effects
@@
 				)
 				(justify left)
-				(hide yes)
 			)
 		)
-		(property "Footprint" "Package_TO_SOT_SMD:SOT-223-3_TabPin2"
-			(at 228.6 48.26 0)
+		(property "Footprint" "Package_TO_SOT_SMD:SOT-23_Handsoldering"
+			(at 233.68 45.72 0)
 			(effects
 				(font
@@
 			)
 		)
-		(property "Description" "Depletion-mode N-channel MOSFET, drain/gate/source"
+		(property "Description" "N-MOSFET transistor, gate/source/drain"
 			(at 228.6 48.26 0)
 			(effects
@@
 	)
 	(symbol
-		(lib_id "Device:Q_NMOS_Depletion_DGS")
+		(lib_id "Device:Q_NMOS_GSD")
 		(at 195.58 82.55 0)
 		(unit 1)
@@
 			)
 		)
-		(property "Value" "Q_NMOS_Depletion_DGS"
+		(property "Value" "AO3400A"
 			(at 201.93 83.8199 0)
 			(effects
@@
 				)
 				(justify left)
-				(hide yes)
 			)
 		)
-		(property "Footprint" "Package_TO_SOT_SMD:SOT-223-3_TabPin2"
-			(at 195.58 82.55 0)
+		(property "Footprint" "Package_TO_SOT_SMD:SOT-23_Handsoldering"
+			(at 200.66 80.01 0)
 			(effects
 				(font
@@
 			)
 		)
-		(property "Description" "Depletion-mode N-channel MOSFET, drain/gate/source"
+		(property "Description" "N-MOSFET transistor, gate/source/drain"
 			(at 195.58 82.55 0)
 			(effects
@@
 	)
 	(symbol
-		(lib_id "Device:Q_NMOS_Depletion_DGS")
+		(lib_id "Device:Q_NMOS_GSD")
 		(at 162.56 48.26 0)
 		(unit 1)
@@
 			)
 		)
-		(property "Value" "Q_NMOS_Depletion_DGS"
+		(property "Value" "AO3400A"
 			(at 168.91 49.5299 0)
 			(effects
@@
 				)
 				(justify left)
-				(hide yes)
 			)
 		)
-		(property "Footprint" "Package_TO_SOT_SMD:SOT-223-3_TabPin2"
-			(at 162.56 48.26 0)
+		(property "Footprint" "Package_TO_SOT_SMD:SOT-23_Handsoldering"
+			(at 167.64 45.72 0)
 			(effects
 				(font
@@
 			)
 		)
-		(property "Description" "Depletion-mode N-channel MOSFET, drain/gate/source"
+		(property "Description" "N-MOSFET transistor, gate/source/drain"
 			(at 162.56 48.26 0)
 			(effects
@@
 	)
 	(symbol
-		(lib_id "Device:Q_NMOS_Depletion_DGS")
+		(lib_id "Device:Q_NMOS_GSD")
 		(at 262.89 48.26 0)
 		(unit 1)
@@
 			)
 		)
-		(property "Value" "Q_NMOS_Depletion_DGS"
+		(property "Value" "AO3400A"
 			(at 269.24 49.5299 0)
 			(effects
@@
 				)
 				(justify left)
-				(hide yes)
 			)
 		)
-		(property "Footprint" "Package_TO_SOT_SMD:SOT-223-3_TabPin2"
-			(at 262.89 48.26 0)
+		(property "Footprint" "Package_TO_SOT_SMD:SOT-23_Handsoldering"
+			(at 267.97 45.72 0)
 			(effects
 				(font
@@
 			)
 		)
-		(property "Description" "Depletion-mode N-channel MOSFET, drain/gate/source"
+		(property "Description" "N-MOSFET transistor, gate/source/drain"
 			(at 262.89 48.26 0)
 			(effects
@@
 	)
 	(symbol
-		(lib_id "Device:Q_NMOS_Depletion_DGS")
+		(lib_id "Device:Q_NMOS_GSD")
 		(at 162.56 82.55 0)
 		(unit 1)
@@
 			)
 		)
-		(property "Value" "Q_NMOS_Depletion_DGS"
+		(property "Value" "AO3400A"
 			(at 168.91 83.8199 0)
 			(effects
@@
 				)
 				(justify left)
-				(hide yes)
 			)
 		)
-		(property "Footprint" "Package_TO_SOT_SMD:SOT-223-3_TabPin2"
-			(at 162.56 82.55 0)
+		(property "Footprint" "Package_TO_SOT_SMD:SOT-23_Handsoldering"
+			(at 167.64 80.01 0)
 			(effects
 				(font
@@
 			)
 		)
-		(property "Description" "Depletion-mode N-channel MOSFET, drain/gate/source"
+		(property "Description" "N-MOSFET transistor, gate/source/drain"
 			(at 162.56 82.55 0)
 			(effects
@@
 	)
 	(symbol
-		(lib_id "Device:Q_NMOS_Depletion_DGS")
+		(lib_id "Device:Q_NMOS_GSD")
 		(at 262.89 82.55 0)
 		(unit 1)
@@
 			)
 		)
-		(property "Value" "Q_NMOS_Depletion_DGS"
+		(property "Value" "AO3400A"
 			(at 269.24 83.8199 0)
 			(effects
@@
 				)
 				(justify left)
-				(hide yes)
 			)
 		)
-		(property "Footprint" "Package_TO_SOT_SMD:SOT-223-3_TabPin2"
-			(at 262.89 82.55 0)
+		(property "Footprint" "Package_TO_SOT_SMD:SOT-23_Handsoldering"
+			(at 267.97 80.01 0)
 			(effects
 				(font
@@
 			)
 		)
-		(property "Description" "Depletion-mode N-channel MOSFET, drain/gate/source"
+		(property "Description" "N-MOSFET transistor, gate/source/drain"
 			(at 262.89 82.55 0)
 			(effects
@@
 	)
 	(symbol
-		(lib_id "Device:Q_NMOS_Depletion_DGS")
+		(lib_id "Device:Q_NMOS_GSD")
 		(at 228.6 82.55 0)
 		(unit 1)
@@
 			)
 		)
-		(property "Value" "Q_NMOS_Depletion_DGS"
+		(property "Value" "AO3400A"
 			(at 234.95 83.8199 0)
 			(effects
@@
 				)
 				(justify left)
-				(hide yes)
 			)
 		)
-		(property "Footprint" "Package_TO_SOT_SMD:SOT-223-3_TabPin2"
-			(at 228.6 82.55 0)
+		(property "Footprint" "Package_TO_SOT_SMD:SOT-23_Handsoldering"
+			(at 233.68 80.01 0)
 			(effects
 				(font
@@
 			)
 		)
-		(property "Description" "Depletion-mode N-channel MOSFET, drain/gate/source"
+		(property "Description" "N-MOSFET transistor, gate/source/drain"
 			(at 228.6 82.55 0)
 			(effects

Commit message: pcb updates
Connections:
- net +3.3V: now also R17.2, R18.2
- net +5VL: no longer R17.2, R18.2
