File: pcb/pubmarine-submarine.kicad_sch (KiCad schematic)
At the start: 97 parts, among them J1 Screw_Terminal_01x02, J10 Conn_01x02, J11 Conn_01x02, J12 Screw_Terminal_01x02, J13 Conn_01x03, J14 Conn_01x04, J15 Servo1, J16 Servo2, J17 Servo3, J18 Servo4, J19 Conn_01x02, J2 Conn_01x02, J20 Conn_01x02, J21 Conn_01x02, J22 Conn_01x02, J23 Conn_01x02, J24 Conn_01x02, J25 Conn_01x20, J26 Conn_01x20, J27 Conn_01x03, J3 Conn_01x02, J4 Conn_01x02, J5 Conn_01x02, J6 Screw_Terminal_01x02, J7 Screw_Terminal_01x02, J8 Conn_01x02, J9 Conn_01x02, Q1 AO3400A, Q2 AO3400A, Q3 AO3400A, Q4 AO3400A, Q5 AO3400A, Q6 AO3400A, Q7 AO3400A, Q8 AO3400A, U1 Pico, U2 SN74LV1T34DBV, U3 A4950E, U4 A4950E, U5 A4950E, U6 A4950E, U7 MPU-6050

Commit message: pcb: fix clearances
Parts:
- J25, J26, J27, JP1: now left out of the parts list
Changed lines of the file:
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@@
 		(unit 1)
 		(exclude_from_sim no)
-		(in_bom yes)
+		(in_bom no)
 		(on_board yes)
 		(dnp no)
@@
 		(unit 1)
 		(exclude_from_sim no)
-		(in_bom yes)
+		(in_bom no)
 		(on_board yes)
 		(dnp no)
@@
 		(unit 1)
 		(exclude_from_sim no)
-		(in_bom yes)
+		(in_bom no)
 		(on_board yes)
 		(dnp no)
@@
 		(unit 1)
 		(exclude_from_sim no)
-		(in_bom yes)
+		(in_bom no)
 		(on_board yes)
 		(dnp no)

Commit message: pcb: fix LSS pins, notes for other rev2 changes
Connections:
- net GND: now also U3.7 (LSS), U4.7 (LSS), U5.7 (LSS), U6.7 (LSS)
- no-connect marks 9 -> 5
Other:
- note added: "TODO revision 2: Change pin mappings so GPIO channels do not conflict"
- note added: "TODO revision 2: LEDs might be too bright?"
- note added: "TODO revision 2: add I2C OLED screen footprint?"
- note added: "TODO revision 2: change to USB-A female?"
- note added: "revision 2: LSS pin is the return path for motor current, must go to ground even when not using RS."

Commit message: pcb v2 wip
Other:
- note added: "TODO revision 2: Change pin mappings so GPIO channels do not conflict Add reset button Change VSYS jumper to default open"
- note removed: "TODO revision 2: Change pin mappings so GPIO channels do not conflict"
Changed lines of the file:
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@@
 		)
 	)
-	(text "TODO revision 2:\nChange pin mappings so GPIO channels do not conflict"
+	(text "TODO revision 2:\nChange pin mappings so GPIO channels do not conflict\nAdd reset button\nChange VSYS jumper to default open"
 		(exclude_from_sim no)
 		(at 104.902 99.06 0)

Commit message: wip: PCB rev2, motors mostly done?
Parts:
- removed C10, C6, C8: 220n, Capacitor_SMD:C_0603_1608Metric_Pad1.08x0.95mm_HandSolder, symbol Device:C
- removed C11, C5, C7, C9: 100u, Capacitor_THT:CP_Radial_D6.3mm_P2.50mm, symbol Device:C_Polarized_US
- removed J19, J20, J21, J22: Conn_01x02, Connector_JST:JST_XH_B2B-XH-AM_1x02_P2.50mm_Vertical, symbol Connector_Generic:Conn_01x02
- removed J27: Conn_01x03, Connector_PinHeader_2.54mm:PinHeader_1x03_P2.54mm_Vertical, symbol Connector_Generic:Conn_01x03
- removed U3, U4, U5, U6: A4950E, Package_SO:SOIC-8-1EP_3.9x4.9mm_P1.27mm_EP2.62x3.51mm_ThermalVias, symbol Driver_Motor:A4950E
- added C18, C19: C, Capacitor_SMD:C_0603_1608Metric_Pad1.08x0.95mm_HandSolder, symbol Device:C
- added C20: 100N, Capacitor_SMD:C_0603_1608Metric_Pad1.08x0.95mm_HandSolder, symbol Device:C
- added J22: Conn_01x04, Connector_PinHeader_2.54mm:PinHeader_1x04_P2.54mm_Vertical, symbol Connector_Generic:Conn_01x04
- added J28, J29: Conn_01x02, Connector_JST:JST_XH_B2B-XH-AM_1x02_P2.50mm_Vertical, symbol Connector_Generic:Conn_01x02
- added Q9: AO3400A, Package_TO_SOT_SMD:SOT-23_Handsoldering, symbol Device:Q_NMOS_GSD
- added R26: 470R, Resistor_SMD:R_0603_1608Metric_Pad0.98x0.95mm_HandSolder, symbol Device:R
- added R27, R31: 10k, Resistor_SMD:R_0603_1608Metric_Pad0.98x0.95mm_HandSolder, symbol Device:R
- added R28: 10K, Resistor_SMD:R_0603_1608Metric_Pad0.98x0.95mm_HandSolder, symbol Device:R
- added SW1: SW_Push, Button_Switch_THT:SW_PUSH_6mm, symbol Switch:SW_Push
- added U5: ER_OLEDM0.91_1x-I2C, Display:ER_OLEDM0.91_1x-I2C, symbol Display_Graphic:ER_OLEDM0.91_1x-I2C
- added U9: ADS1015IDGS, Package_SO:TSSOP-10_3x3mm_P0.5mm, symbol Analog_ADC:ADS1015IDGS
- C1, C2: value 100u -> 220U
- C3: value 100n -> 100N
- C4: value 220n -> 100N
- JP1: value Jumper_2_Bridged -> Jumper_2_Open; footprint Jumper:SolderJumper-2_P1.3mm_Bridged_RoundedPad1.0x1.5mm -> Jumper:SolderJumper-2_P1.3mm_Open_RoundedPad1.0x1.5mm; symbol Jumper:Jumper_2_Bridged -> Jumper:SolderJumper_2_Open
- U1: footprint MCU_RaspberryPi_and_Boards:RPi_Pico_SMD_TH -> pubmarine-submarine:RPi_Pico_SMD_TH; symbol MCU_RaspberryPi_and_Boards:Pico -> pubmarine-submarine:Pico
Connections:
- net +12V: no longer C4.1
- net +3.3V: now also C4.1, J22.1 (Pin_1), R31.2, U5.2 (VCC), U9.8 (VDD)
- net BAT_SENS: no longer J26.9 (Pin_9), U1.32 (GPIO27_ADC1)
- net GND: now also C20.2, J22.3 (Pin_3), Q9.2 (S), R27.2, SW1.2, U5.1 (GND), U9.1 (ADDR), U9.3 (GND); no longer J23.2 (Pin_2), J24.2 (Pin_2), U1.42 (GND)
- net RUN: now also C20.1, R28.1, SW1.1
- net SCL: now also J22.4 (Pin_4), U5.3 (SCL), U9.10 (SCL)
- net SDA: now also J22.2 (Pin_2), U5.4 (SDA), U9.9 (SDA)
- net SENS1: no longer J26.10 (Pin_10), U1.31 (GPIO26_ADC0)
- net VSYS: now reaches J26.2 (Pin_2), JP1.1 (A), U1.39 (VSYS)
- net VSYS: now also R28.2
- net GPIO28_ADC2 renamed ~{FAULT_A}
- net IN_W1: no longer names the net of J25.2 (Pin_2), U1.2 (GPIO1)
- net IN_W2 renamed IN_B2
- net IN_X1: no longer names the net of J26.14 (Pin_14), U1.27 (GPIO21)
- net IN_X2 renamed ~{SLEEP_B}
- net IN_Y1 renamed IN_A1
- net IN_Y2: no longer names the net of J26.15 (Pin_15), U1.26 (GPIO20)
- net IN_Z1 renamed IN_B1
- net IN_Z2 renamed IN_A2
- new net: J23.2 (Pin_2), J24.2 (Pin_2), Q9.3 (D)
- new net: R31.1, U9.2 (ALERT/RDY)
- new net: Q9.1 (G), R26.2, R27.1
- new net A1: C18.1, J28.2 (Pin_2)
- new net A2: C18.2, J28.1 (Pin_1)
- new net B1: C19.1, J29.2 (Pin_2)
- new net B2: C19.2, J29.1 (Pin_1)
- new net LIGHTS: R26.1
- new net ~{FAULT_B}: J26.10 (Pin_10), U1.31 (GPIO26_ADC0)
- new net ~{SLEEP_A}: J26.9 (Pin_9), U1.32 (GPIO27_ADC1)
Other:
- added sheet DRV8873H (DRV8873H.kicad_sch)
- added sheet DRV8873H1 (DRV8873H.kicad_sch)
- note added: "ADS1015 ADC"
- note added: "AHT20 Temp/Humidity"
- note added: "MCU Power and Reset"
- note added: "SSD1306 128x32 OLED"
- note removed: "TODO revision 2: Change pin mappings so GPIO channels do not conflict Add reset button Change VSYS jumper to default open"
- note removed: "TODO revision 2: add I2C OLED screen footprint?"
- note removed: "revision 2: LSS pin is the return path for motor current, must go to ground even when not using RS."

Commit message: wip pcb
Parts:
- removed D1, D2, D3, D4, D5, D6, D7, D8: B5819W, Diode_SMD:D_SOD-123, symbol Device:D_Schottky
- removed J25, J26: Conn_01x20, Connector_PinHeader_2.54mm:PinHeader_1x20_P2.54mm_Vertical, symbol Connector_Generic:Conn_01x20
- removed Q1, Q2, Q3, Q4, Q5, Q6, Q7, Q8: AO3400A, Package_TO_SOT_SMD:SOT-23_Handsoldering, symbol Device:Q_NMOS_GSD
- removed R1, R10, R11, R12, R2, R3, R4, R9: 470R, Resistor_SMD:R_0603_1608Metric_Pad0.98x0.95mm_HandSolder, symbol Device:R
- removed R13, R14, R15, R16, R5, R6, R7, R8: 10k, Resistor_SMD:R_0603_1608Metric_Pad0.98x0.95mm_HandSolder, symbol Device:R
- added C27, C28, C29, C30, C31, C32, C33, C34: C, Capacitor_SMD:C_0603_1608Metric_Pad1.08x0.95mm_HandSolder, symbol Device:C
- added C35, C37: 100N, Capacitor_SMD:C_0603_1608Metric_Pad1.08x0.95mm_HandSolder, symbol Device:C
- added C36, C38: 10U, Capacitor_SMD:C_0603_1608Metric_Pad1.08x0.95mm_HandSolder, symbol Device:C
- added R30, R33: 10k, Resistor_SMD:R_0603_1608Metric_Pad0.98x0.95mm_HandSolder, symbol Device:R
- added U3, U4: DRV8847PWP, Package_SO:HTSSOP-16-1EP_4.4x5mm_P0.65mm_EP3.4x5mm_Mask2.46x2.31mm_ThermalVias, symbol Driver_Motor:DRV8847PWP
- J1, J12, J6, J7: footprint TerminalBlock:TerminalBlock_Altech_AK300-2_P5.00mm -> pubmarine-submarine:TerminalBlock_Altech_AK300-2_P5.00mm
- J28, J29: footprint Connector_JST:JST_XH_B2B-XH-AM_1x02_P2.50mm_Vertical -> pubmarine-submarine:TerminalBlock_Altech_AK300-2_P5.00mm
Connections:
- net FD- is gone; now on net GND: J3.2 (Pin_2)
- net FL- is gone; now on net GND: J4.2 (Pin_2)
- net FR- is gone; now on net GND: J5.2 (Pin_2)
- net FU- is gone; now on net GND: J2.2 (Pin_2)
- net RD- is gone; now on net GND: J9.2 (Pin_2)
- net RL- is gone; now on net GND: J10.2 (Pin_2)
- net RR- is gone; now on net GND: J11.2 (Pin_2)
- net RU- is gone; now on net GND: J8.2 (Pin_2)
- net +12V: now also C1.1, C2.1, C35.1, C36.1, C37.1, C38.1, U3.12 (VM), U4.12 (VM)
- net +3.3V: now also R30.1, R33.1
- net +5VP: no longer C1.1, C2.1, J10.1 (Pin_1), J11.1 (Pin_1), J2.1 (Pin_1), J3.1 (Pin_1), J4.1 (Pin_1), J5.1 (Pin_1), J8.1 (Pin_1), J9.1 (Pin_1)
- net FD: now also U3.15 (IN2)
- net FL: now also U3.10 (IN4)
- net FR: now also U3.9 (IN3)
- net FU: now also U3.16 (IN1)
- net GND: now also C27.2, C28.2, C29.2, C30.2, C31.2, C32.2, C33.2, C34.2, C35.2, C36.2, C37.2, C38.2, U3.11 (TRQ), U3.13 (GND), U3.17 (PPAD), U3.3 (ISEN12), U3.6 (ISEN34), U4.11 (TRQ), U4.13 (GND), U4.17 (PPAD), U4.3 (ISEN12), U4.6 (ISEN34)
- net LIGHTS: now also U1.2 (GPIO1)
- net RD: now also U4.15 (IN2)
- net RL: now also U4.10 (IN4)
- net RR: now also U4.9 (IN3)
- net RU: now also U4.16 (IN1)
- net ADC_VREF: no longer names the net of U1.35 (ADC_VREF)
- net ~{FAULT_A} renamed ~{FAULT_M}
- net ~{FAULT_M}: now also R30.2
- net ~{FAULT_B} renamed ~{FAULT_J}
- net ~{FAULT_J}: now also R33.2, U3.8 (~{FAULT}), U4.8 (~{FAULT})
- net ~{SLEEP_A} renamed ~{SLEEP_M}
- net ~{SLEEP_B} renamed ~{SLEEP_J}
- net ~{SLEEP_J}: now also U3.1 (~{SLEEP}), U4.1 (~{SLEEP})
- new net FD+: C28.1, J3.1 (Pin_1), U3.4 (OUT2)
- new net FL+: C29.1, J4.1 (Pin_1), U3.5 (OUT4)
- new net FR+: C30.1, J5.1 (Pin_1), U3.7 (OUT3)
- new net FU+: C27.1, J2.1 (Pin_1), U3.2 (OUT1)
- new net RD+: C32.1, J9.1 (Pin_1), U4.4 (OUT2)
- new net RL+: C33.1, J10.1 (Pin_1), U4.5 (OUT4)
- new net RR+: C34.1, J11.1 (Pin_1), U4.7 (OUT3)
- new net RU+: C31.1, J8.1 (Pin_1), U4.2 (OUT1)
- no-connect marks 5 -> 11
Other:
- moved on the sheet: J10, J11, J2, J3, J4, J5, J8, J9

Commit message: pcb rev2 done?
Parts:
- C18, C19, C27, C28, C29, C30, C31, C32, C33, C34: value C -> 100N
Connections:
- net BAT_SENS: now also U9.6 (AIN2)
- net IPROPI_A: now also U9.5 (AIN1)
- net IPROPI_B: now also U9.4 (AIN0)
- net SENS1: now also U9.7 (AIN3)
Other:
- moved on the sheet: C4
Changed lines of the file:
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@@
 	(wire
 		(pts
-			(xy 134.62 135.89) (xy 152.4 135.89)
+			(xy 128.27 135.89) (xy 152.4 135.89)
 		)
 		(stroke
@@
 		)
 	)
+	(global_label "BAT_SENS"
+		(shape input)
+		(at 142.24 151.13 180)
+		(effects
+			(font
+				(size 1.27 1.27)
+			)
+			(justify right)
+		)
+		(property "Intersheetrefs" "${INTERSHEET_REFS}"
+			(at 142.24 151.13 0)
+			(hide yes)
+			(show_name no)
+			(do_not_autoplace no)
+			(effects
+				(font
+					(size 1.27 1.27)
+				)
+			)
+		)
+	)
 	(global_label "~{FAULT_J}"
 		(shape input)
@@
 		)
 	)
+	(global_label "SENS1"
+		(shape input)
+		(at 142.24 153.67 180)
+		(effects
+			(font
+				(size 1.27 1.27)
+			)
+			(justify right)
+		)
+		(property "Intersheetrefs" "${INTERSHEET_REFS}"
+			(at 142.24 153.67 0)
+			(hide yes)
+			(show_name no)
+			(do_not_autoplace no)
+			(effects
+				(font
+					(size 1.27 1.27)
+				)
+			)
+		)
+	)
 	(global_label "IN_B1"
 		(shape input)
@@
 		)
 	)
+	(global_label "IPROPI_A"
+		(shape input)
+		(at 142.24 148.59 180)
+		(effects
+			(font
+				(size 1.27 1.27)
+			)
+			(justify right)
+		)
+		(property "Intersheetrefs" "${INTERSHEET_REFS}"
+			(at 142.24 148.59 0)
+			(hide yes)
+			(show_name no)
+			(do_not_autoplace no)
+			(effects
+				(font
+					(size 1.27 1.27)
+				)
+			)
+		)
+	)
 	(global_label "IN_B2"
 		(shape input)
@@
 		)
 	)
+	(global_label "IPROPI_B"
+		(shape input)
+		(at 142.24 146.05 180)
+		(effects
+			(font
+				(size 1.27 1.27)
+			)
+			(justify right)
+		)
+		(property "Intersheetrefs" "${INTERSHEET_REFS}"
+			(at 142.24 146.05 0)
+			(hide yes)
+			(show_name no)
+			(do_not_autoplace no)
+			(effects
+				(font
+					(size 1.27 1.27)
+				)
+			)
+		)
+	)
 	(global_label "RD"
 		(shape input)
@@
 			)
 		)
-		(property "Value" "C"
+		(property "Value" "100N"
 			(at 130.81 259.0799 0)
 			(show_name no)
@@
 			)
 		)
-		(property "Value" "C"
+		(property "Value" "100N"
 			(at 256.54 38.0999 0)
 			(show_name no)
@@
 			)
 		)
-		(property "Value" "C"
+		(property "Value" "100N"
 			(at 223.52 74.9299 0)
 			(show_name no)
@@
 			)
 		)
-		(property "Value" "C"
+		(property "Value" "100N"
 			(at 289.56 74.9299 0)
 			(show_name no)
@@
 			)
 		)
-		(property "Value" "C"
+		(property "Value" "100N"
 			(at 223.52 38.0999 0)
 			(show_name no)
@@
 	(symbol
 		(lib_id "Device:C")
-		(at 134.62 139.7 0)
+		(at 128.27 139.7 0)
 		(mirror y)
 		(unit 1)
@@
 		(dnp no)
 		(property "Reference" "C4"
-			(at 130.81 138.4299 0)
+			(at 124.46 138.4299 0)
 			(show_name no)
 			(do_not_autoplace no)
@@
 		)
 		(property "Value" "100N"
-			(at 130.81 140.9699 0)
+			(at 124.46 140.9699 0)
 			(show_name no)
 			(do_not_autoplace no)
@@
 		)
 		(property "Footprint" "Capacitor_SMD:C_0603_1608Metric_Pad1.08x0.95mm_HandSolder"
-			(at 133.6548 143.51 0)
+			(at 127.3048 143.51 0)
 			(hide yes)
 			(show_name no)
@@
 		)
 		(property "Datasheet" ""
-			(at 134.62 139.7 0)
+			(at 128.27 139.7 0)
 			(hide yes)
 			(show_name no)
@@
 		)
 		(property "Description" "Unpolarized capacitor"
-			(at 134.62 139.7 0)
+			(at 128.27 139.7 0)
 			(hide yes)
 			(show_name no)
@@
 			)
 		)
-		(property "Value" "C"
+		(property "Value" "100N"
 			(at 64.008 258.8259 0)
 			(show_name no)
@@
 			)
 		)
-		(property "Value" "C"
+		(property "Value" "100N"
 			(at 289.56 38.0999 0)
 			(show_name no)
@@
 			)
 		)
-		(property "Value" "C"
+		(property "Value" "100N"
 			(at 256.54 74.9299 0)
 			(show_name no)
@@
 	(symbol
 		(lib_id "power:GND")
-		(at 134.62 143.51 0)
+		(at 128.27 143.51 0)
 		(unit 1)
 		(body_style 1)
@@
 		(fields_autoplaced yes)
 		(property "Reference" "#PWR063"
-			(at 134.62 149.86 0)
+			(at 128.27 149.86 0)
 			(hide yes)
 			(show_name no)
@@
 		)
 		(property "Value" "GND"
-			(at 134.62 148.59 0)
+			(at 128.27 148.59 0)
 			(show_name no)
 			(do_not_autoplace no)
@@
 		)
 		(property "Footprint" ""
-			(at 134.62 143.51 0)
+			(at 128.27 143.51 0)
 			(hide yes)
 			(show_name no)
@@
 		)
 		(property "Datasheet" ""
-			(at 134.62 143.51 0)
+			(at 128.27 143.51 0)
 			(hide yes)
 			(show_name no)
@@
 		)
 		(property "Description" "Power symbol creates a global label with name \"GND\" , ground"
-			(at 134.62 143.51 0)
+			(at 128.27 143.51 0)
 			(hide yes)
 			(show_name no)
@@
 			)
 		)
-		(property "Value" "C"
+		(property "Value" "100N"
 			(at 323.85 74.9299 0)
 			(show_name no)
@@
 			)
 		)
-		(property "Value" "C"
+		(property "Value" "100N"
 			(at 323.85 38.0999 0)
 			(show_name no)

Commit message: pcb tweaks
Parts:
- R17, R18: value 4k7 -> 2k2
Other:
- note added: "TODO: - Review analog signal lines - Break out extra GPIOs - Break out RST pin (wire to Pi) - Add stitching vias - Review datasheets - Schematic cleanup - Fix silkscreen graphics - Design review - Add BOM/CPL - Ship it"
Changed lines of the file:
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@@
 		)
 	)
+	(text "TODO:\n- Review analog signal lines\n- Break out extra GPIOs\n- Break out RST pin (wire to Pi)\n- Add stitching vias\n- Review datasheets\n- Schematic cleanup\n- Fix silkscreen graphics\n- Design review\n- Add BOM/CPL\n- Ship it\n"
+		(exclude_from_sim no)
+		(at 277.368 149.098 0)
+		(effects
+			(font
+				(size 1.27 1.27)
+				(color 255 0 0 1)
+			)
+			(justify left)
+		)
+	)
 	(text "IMU Module"
 		(exclude_from_sim no)
@@
 			)
 		)
-		(property "Value" "4k7"
+		(property "Value" "2k2"
 			(at 176.53 204.4699 0)
 			(show_name no)
@@
 			)
 		)
-		(property "Value" "4k7"
+		(property "Value" "2k2"
 			(at 166.37 204.4699 0)
 			(show_name no)

Commit message: pcb updates
Parts:
- added C5, C6: 100N, Capacitor_SMD:C_0603_1608Metric_Pad1.08x0.95mm_HandSolder, symbol Device:C
- added J19: Conn_01x03_Pin, Connector_PinHeader_2.54mm:PinHeader_1x03_P2.54mm_Vertical, symbol Connector:Conn_01x03_Pin
- added J20: Conn_01x02_Pin, Connector_PinHeader_2.54mm:PinHeader_1x02_P2.54mm_Vertical, symbol Connector:Conn_01x02_Pin
- added TP1, TP2: TestPoint, TestPoint:TestPoint_Pad_D1.0mm, symbol Connector:TestPoint
- J15: value Servo1 -> Conn_01x03
- J16: value Servo2 -> Conn_01x03
- J17: value Servo3 -> Conn_01x03
- J18: value Servo4 -> Conn_01x03
- J28, J29: value Conn_01x02 -> Screw_Terminal_01x02; symbol Connector_Generic:Conn_01x02 -> Connector:Screw_Terminal_01x02
- R28: value 10K -> 10k
Connections:
- net +3.3V: now also U7.1 (VCC), C6.1
- net +5VL: now also C5.1; no longer U7.1 (VCC)
- net GND: now also C5.2, C6.2, J19.1 (Pin_1), J20.1 (Pin_1)
- net IPROPI_A: now also TP1.1
- net IPROPI_B: now also TP2.1
- net RUN: now also J20.2 (Pin_2)
- net ~{FAULT_J}: now also U1.27 (GPIO21); no longer U1.31 (GPIO26_ADC0)
- net ~{SLEEP_J}: now also U1.26 (GPIO20); no longer U1.29 (GPIO22)
- net ~{SLEEP_M}: now also U1.29 (GPIO22); no longer U1.32 (GPIO27_ADC1)
- new net: J19.3 (Pin_3), U1.31 (GPIO26_ADC0)
- new net: J19.2 (Pin_2), U1.32 (GPIO27_ADC1)
- no-connect marks 11 -> 9
Other:
- note removed: "TODO revision 2: LEDs might be too bright?"
- note removed: "TODO revision 2: change to USB-A female?"
- note removed: "TODO: - Review analog signal lines - Break out extra GPIOs - Break out RST pin (wire to Pi) - Add stitching vias - Review datasheets - Schematic cleanup - Fix silkscreen graphics - Design review - Add BOM/CPL - Ship it"
