File: pcb/DRV8873H.kicad_sch (KiCad schematic)
At the start: 11 parts, among them U10 DRV8873H

Commit message: wip pcb
Parts:
- removed R30: 10K, Resistor_SMD:R_0603_1608Metric_Pad0.98x0.95mm_HandSolder, symbol Device:R
