File: pcb/DRV8873H.kicad_block/DRV8873H.kicad_pcb (KiCad board)
At the start: 4 copper layers, 11 parts, among them U10 DRV8873H

Commit message: wip pcb
Parts:
- removed C12, C14: 1U, Capacitor_SMD:C_0603_1608Metric_Pad1.08x0.95mm_HandSolder
- removed C13, C15: 100N, Capacitor_SMD:C_0603_1608Metric_Pad1.08x0.95mm_HandSolder
- removed C16: 47N, Capacitor_SMD:C_0603_1608Metric_Pad1.08x0.95mm_HandSolder
- removed C17: 220U, Capacitor_THT:CP_Radial_D6.3mm_P2.50mm
- removed JP2, JP3: SolderJumper_3_Bridged12, Jumper:SolderJumper-3_P1.3mm_Bridged12_RoundedPad1.0x1.5mm
- removed R29: 330R, Resistor_SMD:R_0603_1608Metric_Pad0.98x0.95mm_HandSolder
- removed R30: 10K, Resistor_SMD:R_0603_1608Metric_Pad0.98x0.95mm_HandSolder
- removed U10: DRV8873H, Package_SO:HTSSOP-24-1EP_4.4x7.8mm_P0.65mm_EP3.4x7.8mm_Mask2.44x3.42mm_ThermalVias
- added C19: C, Capacitor_SMD:C_0603_1608Metric_Pad1.08x0.95mm_HandSolder, F.Cu at (93.5, 54.2)
- added C21: 1U, Capacitor_SMD:C_0603_1608Metric_Pad1.08x0.95mm_HandSolder, F.Cu at (87.2, 63.5)
- added C22: 100N, Capacitor_SMD:C_0603_1608Metric_Pad1.08x0.95mm_HandSolder, F.Cu at (97.2, 59.2)
- added C23: 1U, Capacitor_SMD:C_0603_1608Metric_Pad1.08x0.95mm_HandSolder, F.Cu at (87.0, 55.0)
- added C24: 100N, Capacitor_SMD:C_0603_1608Metric_Pad1.08x0.95mm_HandSolder, F.Cu at (85.5, 55.0)
- added C25: 47N, Capacitor_SMD:C_0603_1608Metric_Pad1.08x0.95mm_HandSolder, F.Cu at (87.0, 58.5)
- added JP4: SolderJumper_3_Bridged12, Jumper:SolderJumper-3_P1.3mm_Bridged12_RoundedPad1.0x1.5mm, B.Cu at (89.7, 66.2)
- added JP5: SolderJumper_3_Bridged12, Jumper:SolderJumper-3_P1.3mm_Bridged12_RoundedPad1.0x1.5mm, B.Cu at (93.4, 66.2)
- added R32: 330R, Resistor_SMD:R_0603_1608Metric_Pad0.98x0.95mm_HandSolder, F.Cu at (97.2, 63.6)
- added U11: DRV8873H, Package_SO:HTSSOP-24-1EP_4.4x7.8mm_P0.65mm_EP3.4x7.8mm_Mask2.44x3.42mm_ThermalVias, F.Cu at (92.2, 61.2)
Routing:
- net /DRV8873H/DVDD: track 20.0 -> 0.00 mm, vias 2 -> 0
- net /DRV8873H1/DVDD: track 0.00 -> 13.8 mm, vias 0 -> 2
- net IN_A1: track 9.79 -> 0.00 mm
- net IN_A2: track 9.20 -> 0.00 mm
- net IPROPI_B: track 0.00 -> 7.36 mm
- net /A1: track 7.18 -> 0.00 mm
- net IPROPI_A: track 6.86 -> 0.00 mm
- net ~{FAULT_A}: track 6.83 -> 0.00 mm
- net /A2: track 5.97 -> 0.00 mm
- net Net-(U11-VCP): track 0.00 -> 5.08 mm
- net GND: track 23.1 -> 18.3 mm, vias 1 -> 0
- net Net-(U11-CPH): track 0.00 -> 4.63 mm
- net Net-(U11-CPL): track 0.00 -> 4.49 mm
- net ~{FAULT_M}: track 0.00 -> 4.33 mm
- net Net-(U10-CPL): track 3.52 -> 0.00 mm
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- added copper zone on F.Cu, net +12V
